Commit message: add controller, fix gazebo

File: src/robot_description/urdf/lidar.xacro (robot description, xacro)
@@ -7,6 +7,5 @@
         <visual>
             <geometry>
-                <mesh filename="file://$(find robot_description)/mesh/sensors/lds.stl"/>
-                <!-- <mesh filename="file://$(xacro:find-pkg-share robot_description)/mesh/sensors/lds.stl" scale="0.001 0.001 0.001"/> -->
+                <mesh filename="file:///home/thien123/ROS2WS/robocon_ws/install/robot_description/share/robot_description/mesh/sensors/lds.stl" scale="0.001 0.001 0.001"/>
             </geometry>
             <origin xyz="0 0 ${lidar_height/4}" rpy="0 0 0" />
@@ -26,5 +25,5 @@
         <origin xyz="0 0 ${base_height}" rpy="0 0 0" />
     </joint>
-    <!-- <gazebo reference="laser_link">
+    <gazebo reference="laser_link">
         <sensor name="laser" type="ray">
             <pose> 0 0 0 0 0 0 </pose>
@@ -54,4 +53,4 @@
             </plugin>
         </sensor>
-    </gazebo> -->
+    </gazebo>
 </robot>

File: src/robot_description/urdf/my_robot.urdf (robot description, URDF)
Before this commit: robot thien_robot, 7 links, 6 joints
Links:
- link caster_wheel_link: mass 5.0 -> 2.0
Joints:
- joint base_caster_wheel_joint: origin xyz=0.09999999999999999 0 -0.025 rpy=0 0 0 -> xyz=0.1 0 -0.025 rpy=0 0 0; type fixed -> continuous
