Commit message: Modified files

File: src/robot_description/urdf/camera.xacro (robot description, xacro)
@@ -24,14 +24,3 @@
         <origin xyz="${(base_length + camera_length)/2.0 } 0 ${base_height/2.0}" rpy="0 0 0" />
     </joint>
-    <!-- <gazebo reference="camera_link">
-        <material>Gazebo/Red</material>
-        <sensor name="camera_sensor" type="camera">
-            <pose>0 0 0 0 0 0</pose>
-            <visualize>true</visualize>
-            <update_rate>10.0</update_rate>
-            <plugin name="plugin_name" filename="libgazebo_ros_camera.so">
-                <frame_name>camera_link</frame_name>
-            </plugin>
-        </sensor>
-    </gazebo> -->
 </robot>

File: src/robot_description/urdf/lidar.xacro (robot description, xacro)
@@ -25,32 +25,3 @@
         <origin xyz="0 0 ${base_height}" rpy="0 0 0" />
     </joint>
-    <gazebo reference="laser_link">
-        <sensor name="laser" type="ray">
-            <pose> 0 0 0 0 0 0 </pose>
-            <visualize>true</visualize>
-            <update_rate>10.0</update_rate>
-            <ray>
-                <scan>
-                    <horizontal>
-                        <sample>720</sample>
-                        <resolution>1</resolution>
-                        <min_angle>-3.14</min_angle>
-                        <max_angle>3.14</max_angle>
-                    </horizontal>
-                </scan>
-                <range>
-                    <min>0.5</min>
-                    <max>18.0</max>
-                    <resolution>1</resolution>
-                </range>
-            </ray>
-            <plugin name="laser_controller" filename="libgazebo_ros_ray_sensor.so">
-                <ros>
-                    <argument>~/out:=scan</argument>
-                </ros>
-                <output_type>sensor_msgs/LaserScan</output_type>
-                <frame_name>laser_link</frame_name>
-            </plugin>
-        </sensor>
-    </gazebo>
 </robot>

File: src/robot_description/urdf/my_robot.urdf (robot description, URDF)
Before this commit: robot thien_robot, 7 links, 6 joints
Links:
- link caster_wheel_link: mass 2.0 -> 5.0
Joints:
- joint base_caster_wheel_joint: axis 0 1 0 -> 0 1 1; origin xyz=0.1 0 -0.025 rpy=0 0 0 -> xyz=0.09999999999999999 0 -0.025 rpy=0 0 0

File: src/robot_description/urdf/my_robot.urdf.xacro (robot description, xacro)
@@ -5,3 +5,4 @@
     <xacro:include filename="lidar.xacro"/>
     <xacro:include filename="camera.xacro"/>
+    <xacro:include filename="gazebo.xacro"/>
 </robot>

File: src/robot_description/urdf/robot_base.xacro (robot description, xacro)
@@ -105,9 +105,9 @@
         <axis xyz="0 1 0" />
     </joint>
-    <joint name="base_caster_wheel_joint" type="fixed">
+    <joint name="base_caster_wheel_joint" type="continuous">
         <parent link="base_link" />
         <child link="caster_wheel_link" />
         <origin xyz="${base_length / 3.0} 0 ${-wheel_radius / 2.0}" rpy="0 0 0" />
-        <axis xyz="0 1 0" />
+        <axis xyz="0 1 1" />
     </joint>
 </robot>
